Commit message: Fix calibration offset

File: niryo_robot_description/urdf/ned2/niryo_ned2_param.urdf.xacro (robot description, xacro)
@@ -5,6 +5,6 @@
     <!-- Properties -->
     <xacro:property name="distance_hand_tool" value="0.0285"/>
-    <xacro:property name="limit_low_shoulder_rotation" value="-169.03"/>
-    <xacro:property name="limit_up_shoulder_rotation" value="169.03"/>
+    <xacro:property name="limit_low_shoulder_rotation" value="-171.88"/>
+    <xacro:property name="limit_up_shoulder_rotation" value="171.88"/>
     <xacro:property name="limit_low_arm_rotation" value="-105.0"/>
     <xacro:property name="limit_up_arm_rotation" value="34.96"/>
